File: hardware/jaladarangam-control-board/jaladarangam-control-board.kicad_pcb (KiCad board)
At the start: 2 copper layers, 145 x 110 mm, 47 parts, among them J1 RPi_GPIO_2x20, J10 MOTOR0, J11 MOTOR1, J12 MOTOR2, J13 MOTOR3, J14 MOTOR4, J15 MOTOR5, J16 MOTOR6, J17 MOTOR7, J18 MOTOR_PWR, J19 AUX_IN, J2 FSR0, J3 FSR1, J4 FSR2, J5 FSR3, J6 FSR4, J7 FSR5, J8 FSR6, J9 FSR7, U1 MCP3008, U2 74HC595, U3 ULN2803A, U4 74HC165

Commit message: Mark J18 polarity on silkscreen, and fix a module ordering bug
Adds "+" and "GND" to the silkscreen above the motor supply input,
each centred over the pad it labels. J18 carries a separate, possibly
higher-voltage rail, and connecting it backwards would drive MOTOR_V+
straight onto the board's ground net; the pad-1 square marker alone did
not say which pin was which.

The change is silkscreen-only in electrical terms - J18's pads stay at
(124.50, 92.00) and (119.50, 92.00), the footprint is untouched and no
copper moved. It was still routed through board_spec.py and the full
pipeline rather than patched into the .kicad_pcb, because gen_pcb.py
rebuilds the board from the spec on every run and a manual edit would
be erased by the next build.

Also moves the "MOTOR PWR" caption clear of the terminal block's body
outline, which it had been overlapping, via a per-connector caption gap.

board_spec.sanity_check now cross-checks every polarity mark against the
net actually on that pad, so a future net change cannot leave a stale
and actively misleading label on a power connector. Verified by flipping
the two marks and confirming both are rejected.

Fixes a latent bug found while adding that check: the module's
__main__ block had been left mid-file when the PCB layout tables were
appended below it, so running board_spec.py directly raised NameError on
names defined further down. Moved to the end of the file.

Re-verified after a full regeneration and re-route:
* ERC: 0 violations
* Netlist cross-check: 45/45 nets match board_spec pad-for-pad
* Net classes: 0.8 mm Power / 0.4 mm signal intact through project,
  board, DSN and laid copper
* Routing: 0 unrouted, 0 violations (433 items, 13 vias)
* DRC on the routed board: 0 violations, 0 unconnected, and no
  silkscreen-clearance violations from the new text
* Zone separation: motor and analog copper still in their own zones

Gerbers, drill files, BOMs and review images regenerated. schematic.pdf
was left alone: the schematic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
Routing:
- net SPI_MOSI: track 88.1 -> 114.5 mm, vias 2 -> 1
- net SPI_MISO: track 89.0 -> 112.5 mm, vias 2 -> 1
- net MOTOR1: track 48.2 -> 64.7 mm
- net MTRDRV7: track 43.1 -> 28.6 mm, vias 1 -> 0
- net MOTOR0: track 54.3 -> 67.7 mm
- net SR_SRCLK: track 135.7 -> 147.4 mm
- net IN_QH: track 62.0 -> 73.6 mm, vias 0 -> 2
- net MTRDRV6: track 26.5 -> 37.5 mm
- net FSR7: track 50.2 -> 61.0 mm, vias 1 -> 0
- net SPI_SCLK: track 103.8 -> 95.0 mm
- net IN_SHLD: track 77.0 -> 69.8 mm, vias 2 -> 1
- net MTRDRV1: track 26.5 -> 32.4 mm
- net MOTOR5: track 41.3 -> 36.9 mm
- net GND: track 562.1 -> 558.2 mm
- net AUX6: track 42.5 -> 38.7 mm
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Other:
- board text added: "+"
- board text added: "GND"

Commit message: Mark motor header polarity, and verify marks against placed pads
Adds "+" and "-" to the silkscreen at J10-J17, in the clear board margin
outboard of each pad: "+" beside pin 1 on MOTOR_V+, "-" beside pin 2 on
that channel's ULN2803A output. Their pins stack 2.54 mm apart, too
close to caption from above the way J18's side-by-side pins are, so the
marks go outboard instead.

This completes the polarity marking started at J18. Every pin carrying
MOTOR_V+ off the board is now identified, so a motor or supply cannot be
wired backwards by reading the board alone.

Verified the silk does not contradict itself: pad 1 is the rectangular
pad with the footprint's L-shaped pin-1 corner beside it, and "+" sits
next to that same pad. The box around pad 2 in a silkscreen-only view is
the connector body outline, not a second pin-1 marker.

Checking the marks, in two independent layers
---------------------------------------------
The polarity table now states, per entry, which net it asserts is on
that pad, and board_spec.sanity_check enforces it against the netlist.
Tested by mutation - three deliberate faults, all rejected:
  * J10's two marks swapped (motor wired backwards)
  * J11 pin 2 claiming MOTOR0 rather than MOTOR1 (off-by-one across
    eight near-identical headers)
  * J17 pin 1 claiming GND rather than MOTOR_V+

That only proves the table is self-consistent, so verify_polarity.py
adds a second check on the generated board: for each mark it finds the
placed silkscreen text, finds the pad nearest to it, and requires that
pad to be the one named and to carry the asserted net. A mark can be
right in the table and still land closer to the neighbouring pin, which
on a 2.54 mm header would tell an assembler to reverse a motor. Tested
by nudging J10's "+" down 2.54 mm on a scratch board and confirming it
is rejected:

  '+' mark for J10 pad 1 sits nearest J10 pad 2 (MOTOR0) instead

It now runs as step 6 of build.sh, so all 18 marks are checked on every
build.

Re-verified a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
Routing:
- net SPI_MOSI: track 114.5 -> 89.7 mm, vias 1 -> 2
- net MOTOR1: track 64.7 -> 48.2 mm
- net FSR7: track 61.0 -> 44.9 mm, vias 0 -> 1
- net MOTOR0: track 67.7 -> 54.3 mm
- net MOTOR7: track 43.1 -> 55.5 mm, vias 0 -> 1
- net SPI_MISO: track 112.5 -> 100.6 mm, vias 1 -> 2
- net SPI_CE0: track 55.8 -> 65.0 mm
- net +3V3: track 331.0 -> 339.8 mm
- net GND: track 558.2 -> 566.5 mm
- net IN_SHLD: track 69.8 -> 61.6 mm
- net SR_RCLK: track 125.2 -> 132.9 mm, vias 2 -> 1
- net MTRDRV6: track 37.5 -> 30.7 mm
- net SR_SRCLK: track 147.4 -> 141.4 mm
- net SPI_SCLK: track 95.0 -> 100.8 mm, vias 0 -> 2
- net MTRDRV2: track 26.5 -> 30.8 mm
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Other:
- board text added: "-"
